Commit message: reorganization of files

File: rudis_magic_sawyer.urdf (robot description, URDF)
Before this commit: robot sawyer, 33 links, 32 joints
Links:
- link head: geometry collision sphere radius=0.18; visual mesh filename=//u/teddy/Robotics_Research/catkin_ws/src/sawyer_robot-mast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
- link pedestal: geometry collision cylinder length=0.62 radius=0.18; visual mesh filename=/u/teddy/Robotics_Research/catkin_ws/src/sawyer_robot-maste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
- link right_arm_base_link: geometry collision cylinder length=0.24 radius=0.08; visual mesh filename=/u/teddy/Robotics_Research/catkin_ws/src/sawyer_robot-maste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
- link right_connector_plate_base: geometry collision cylinder length=0.0302 radius=0.04; visual mesh filename=/u/teddy/Robotics_Research/catkin_ws/src/intera_common-mast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
- link right_electric_gripper_base: geometry collision cylinder length=0.1 radius=0.029; visual mesh filename=/u/teddy/Robotics_Research/catkin_ws/src/intera_common-mast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
- link right_gripper_l_finger: geometry collision box size=0.01 0.0135 0.075; collision box size=0.01 0.05 0.017
- link right_gripper_l_finger_tip: geometry collision box size=0.016 0.007 0.037; visual mesh filename=/u/teddy/Robotics_Research/catkin_ws/src/intera_common-mast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
- link right_gripper_r_finger: geometry collision box size=0.01 0.0135 0.075; collision box size=0.01 0.05 0.017
- link right_gripper_r_finger_tip: geometry collision box size=0.016 0.007 0.037; visual mesh filename=/u/teddy/Robotics_Research/catkin_ws/src/intera_common-mast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
- link right_l0: geometry collision sphere radius=0.07; visual mesh filename=/u/teddy/Robotics_Research/catkin_ws/src/sawyer_robot-maste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
- link right_l1: geometry collision sphere radius=0.07; visual mesh filename=/u/teddy/Robotics_Research/catkin_ws/src/sawyer_robot-maste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
- link right_l2: geometry collision cylinder length=0.34 radius=0.06; visual mesh filename=/u/teddy/Robotics_Research/catkin_ws/src/sawyer_robot-maste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
- link right_l3: geometry collision sphere radius=0.06; visual mesh filename=/u/teddy/Robotics_Research/catkin_ws/src/sawyer_robot-maste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
- link right_l4: geometry collision cylinder length=0.30 radius=0.045; visual mesh filename=/u/teddy/Robotics_Research/catkin_ws/src/sawyer_robot-maste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
- link right_l5: geometry collision sphere radius=0.06; visual mesh filename=/u/teddy/Robotics_Research/catkin_ws/src/sawyer_robot-maste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
- link right_l6: geometry collision cylinder length=0.05 radius=0.055; visual mesh filename=/u/teddy/Robotics_Research/catkin_ws/src/sawyer_robot-maste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
